File: hardware/V0.4/Controller/Controller-PowerSupply.sch (KiCad schematic (older format))
At the start: 22 parts

Commit message: Started work on uController
Parts:
- removed C?: 100n, IPC7351-Nominal:CAPC1608X55, symbol C-0603
- removed C?: 2.2u, IPC7351-Nominal:CAPC2012X70, symbol C-0805
- removed C?: 10n, IPC7351-Nominal:CAPC1608X55, symbol C-0603
- removed D?: B340A-13-F, Diodes-SMD:SMA, symbol B340A-13-F
- removed L?: 784770470-WURTH, manuf:784770470, symbol L-784770470-WURTH
- removed R?: 10k, IPC7351-Nominal:RESC1608X50, symbol R-0603
- removed R?: 1k13, IPC7351-Nominal:RESC1608X50, symbol R-0603
- removed U?: TPS5430DDA, IPC7351-Nominal:SO-8, symbol TPS5430DDA
- added C? (x6): 10uF, IPC7351-Nominal:CAPC1608X55, symbol C-0603
- added C? (x2): 0.1uF, IPC7351-Nominal:CAPC1608X55, symbol C-0603
- added D? (x2): RB168L-40TE25CT-ND, symbol SCHOTTKY
- added L?: 100uH, manuf:BOURNS-SRR7045, symbol L-BOURNS-SRR7045
- added L?: L-BOURNS-SRR7045, manuf:BOURNS-SRR7045, symbol L-BOURNS-SRR7045
- added R?: 84K, IPC7351-Nominal:RESC2012X50, symbol R-0805
- added R?: 6K, IPC7351-Nominal:RESC2012X50, symbol R-0805
- added R? (x2): R-0805, IPC7351-Nominal:RESC2012X50, symbol R-0805
- added U? (x2): AOZ1282, smd-semi:SOT-23-6, symbol AOZ1282
Connections:
- net +12V: now also C?.1, C?.1, C?.1, L?.1, R?.1, U?.4 (EN), U?.5 (VIN)
- net +5V: now also C?.1, L?.1, R?.1
- net GND: now also C?.2, C?.2, C?.2, C?.2, C?.2, C?.2, D?.2 (A), D?.2 (A), R?.2, R?.2, U?.2 (GND), U?.2 (GND)
- net VIN: now also C?.1, C?.1, U?.4 (EN), U?.5 (VIN)
- new net: C?.1, U?.1 (BST) (x2)
- new net: R?.1, R?.2, U?.3 (FB) (x2)
- new net: C?.2, D?.1 (K), L?.3, U?.6 (LX) (x2)
- no-connect marks 1 -> 0
Other:
- moved on the sheet: C?, J?, U?

Commit message: Continued work on the power supply and controller board
Parts:
- removed R?: 84K, IPC7351-Nominal:RESC2012X50, symbol R-0805
- removed R?: 6K, IPC7351-Nominal:RESC2012X50, symbol R-0805
- added R1: 140K, IPC7351-Nominal:RESC1608X50, symbol R-0603
- added R2: 10K, IPC7351-Nominal:RESC1608X50, symbol R-0603
- C1: renamed from C?; value 10uF -> 6u8/50V; footprint IPC7351-Nominal:CAPC1608X55 -> IPC7351-Nominal:CAPC3216X90; PN (none) -> C3216X5R1H685K160AB
- C10, C12: renamed from C?; value 100n -> 100n/16V
- C11: renamed from C?; value 0.1uF -> 100n/16V
- C13: renamed from C?; value 2u2/16V -> 2u2/10V; PN (none) -> CL10A225KP8NNNC
- C14, C7: renamed from C?; value 10uF -> 1uF; PN (none) -> GRM188R61C105KA93D
- C2: renamed from C?; value 10uF -> DNP; footprint IPC7351-Nominal:CAPC1608X55 -> IPC7351-Nominal:CAPC3216X90
- C3, C5: renamed from C?; footprint pth-passive:C-ALUM-16mm -> pth-passive:C-ALUM-8mm; symbol C-ALUM-16mm -> C-ALUM-8mm
- C4: renamed from C?; value 0.1uF -> 100n/50V
- C6: renamed from C?; value 10uF -> 10u/16V; footprint IPC7351-Nominal:CAPC1608X55 -> IPC7351-Nominal:CAPC3216X90; PN (none) -> CL31F106ZOHNNNE
- C8: renamed from C?; PN (none) -> CL10A475KO8NNNC
- C9: renamed from C?; value 10uF -> DNP
- J2: renamed from J?; value CONN-100MIL-M-1x4-SHROUD -> EXT_POWER
- L1: renamed from L?; footprint manuf:BOURNS-SRR7045 -> manuf:BOURNS-SRN8040; symbol L-BOURNS-SRR7045 -> L-BOURNS-SRN8040; Digikey PN# L-BOURNS-SRR7045 -> (none); PN (none) -> SRN8040-101M
- L2: renamed from L?; value L-BOURNS-SRR7045 -> 330uF; footprint manuf:BOURNS-SRR7045 -> manuf:BOURNS-SRN1060; symbol L-BOURNS-SRR7045 -> L-BOURNS-SRN1060; PN (none) -> SRN1060-331M
- R3: renamed from R?; value R-0805 -> 52.3K; PN (none) -> RMCF0603FT52K3
- R4: renamed from R?; value R-0805 -> 10K
- U1, U2: renamed from U?; PN (none) -> AOZ1282CI
- U3: renamed from U?; footprint (none) -> smd-semi:SOT-23; symbol VREG_FIXED -> MCP1700T-vv02E/TT; PN (none) -> MCP1702T-5002E/CB
- gave numbers to parts that had none: 8
Connections:
- net +12V: now also U3.3 (IN), R1.1; no longer U3.IN
- net +5V: now also U3.2 (OUT); no longer U3.OUT
- net EGND: now also C1.2, C10.2, C12.2, C13.2, C14.2, C2.2, C3.2, C5.2, C6.2, C7.2, C8.2, C9.2, D1.1 (-), D2.2 (A), D3.2 (A), J2.2, J2.3, P5.1 (P1), R4.2, U1.2 (GND), U2.2 (GND), U3.1, R2.2
- net at U1.3 (FB): now also R1.2, R2.1
- removed net GND: C1.2, C10.2, C12.2, C13.2, C14.2, C2.2, C3.2, C5.2, C6.2, C7.2, C8.2, C9.2, D1.1 (-), D2.2 (A), D3.2 (A), J2.2, J2.3, P5.1 (P1), R4.2, U1.2 (GND), U2.2 (GND), U3.GND
Other:
- note added: "Populate one or the other 5V section"
- moved on the sheet: C1, C10, C11, C12, C13, C14, C2, C3, C4, C5, C6, C7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
