File: hardware/V0.4/Controller/Controller-uController.sch (KiCad schematic (older format))
At the start: 8 parts

Commit message: Continued work on the power supply and controller board
Parts:
- added C19, C20: 100n/16V, IPC7351-Nominal:CAPC1608X55, symbol C-0603
- added D4: 1N4001, pth-semi:DO-41, symbol 1N4001
- added D5, D6: 1N4148, symbol DIODE
- added D7: Z5.6, symbol DIODE
- added J4: TTL-232R-5V ONLY!, conn-100mil:CONN-100MIL-M-1x6, symbol CONN-100MIL-M-1x6
- added J5: ISP, conn-100mil:CONN-100MIL-M-2x3, symbol CONN-100MIL-M-2x3
- added J6: KEYPAD, conn-100mil:CONN-100MIL-M-1x8, symbol CONN-100MIL-M-1x8
- added Q1: PMOS, symbol PMOS
- added R10, R11: ???, IPC7351-Nominal:RESC1608X50, symbol R-0603
- added R5, R7, R9: 10K, IPC7351-Nominal:RESC1608X50, symbol R-0603
- added R8: 1K, IPC7351-Nominal:RESC1608X50, symbol R-0603
- added RV1, RV2: 10K, symbol POT
- C15, C16, C17, C18: renamed from C?; value 0.1uF -> 100n/16V
- gave numbers to parts that had none: 4
Connections:
- net +5V: now also D4.1 (K), J5.2, Q1.3 (S), R5.1, R7.2, R9.1; no longer J3.15, J3.16
- net BUSY: now also U4.14 (PCINT29/OC1A/PD5); no longer U4.15 (PCINT30/OC2B/ICP/PD6)
- net GND: now also C19.2, C20.2, D7.2 (A), J4.1, J5.6, J6.2
- net Sin/Test: now also U4.11 (PCINT26/RXD1/PD2); no longer U4.12 (PCINT27/TXD1/INT1/PD3)
- net ~CS~: now also U4.12 (PCINT27/TXD1/INT1/PD3); no longer U4.13 (PCINT28/XCK/OC1B/PD4)
- net ~WR~: now also U4.13 (PCINT28/XCK/OC1B/PD4); no longer U4.14 (PCINT29/OC1A/PD5)
- net MOSI: now reaches U4.1 (PCINT13/MOSI/PB5)
- net MOSI: now also J5.4
- net TXD: now reaches U4.10 (PCINT25/TXD0/PD1)
- net TXD: now also J4.5
- net POWER_SWITCH: now reaches U4.16 (PCINT31/OC2A/PD7)
- net POWER_SWITCH: now also J6.1, R9.2
- net MISO: now reaches U4.2 (PCINT14/MISO/PB6)
- net MISO: now also J5.1
- net SCK: now reaches U4.3 (PCINT15/SCK/PB7)
- net SCK: now also J5.3
- net V_REVERSE: now reaches U4.30 (PCINT7/ADC7/PA7)
- net V_REVERSE: now also C20.1
- net V_FOWARD: now reaches U4.31 (PCINT6/ADC6/PA6)
- net V_FOWARD: now also C19.1
- net KEYPAD_ROW_3: now reaches U4.32 (PCINT5/ADC5/PA5)
- net KEYPAD_ROW_3: now also J6.8
- net KEYPAD_ROW_2: now reaches U4.33 (PCINT4/ADC4/PA4)
- net KEYPAD_ROW_2: now also J6.7
- net KEYPAD_ROW_1: now reaches U4.34 (PCINT3/ADC3/PA3)
- net KEYPAD_ROW_1: now also J6.6
- net KEYPAD_COL_3: now reaches U4.35 (PCINT2/ADC2/PA2)
- net KEYPAD_COL_3: now also J6.5
- net KEYPAD_COL_2: now reaches U4.36 (PCINT1/ADC1/PA1)
- net KEYPAD_COL_2: now also J6.4
- net KEYPAD_COL_1: now reaches U4.37 (PCINT0/ADC0/PA0)
- net KEYPAD_COL_1: now also J6.3
- net ~RESET~: now reaches R6.2, U4.4 (~RESET~)
- net ~RESET~: now also J5.5
- net VLIM_OUT: now reaches U4.41 (T1/CLKO/PCINT9/PB1)
- net VLIM_OUT: now also D5.2 (A), D6.1 (K)
- net TIP_DETECT: now reaches U4.42 (AIN0/INT2/PCINT10/PB2)
- net TIP_DETECT: now also R7.1
- net at U4.43 (AIN1/OC0A/PCINT11/PB3): now also R8.2
- net RXD: now reaches U4.9 (PCINT24/RXD0/PD0)
- net RXD: now also J4.4
- new net: J3.15, J3.16, Q1.2 (D)
- new net: D4.2 (A), J4.3
- new net: D5.1 (K), R10.2
- new net: D6.2 (A), R11.2
- new net: R10.1, RV1.3
- new net: R11.1, RV2.3
- new net DISPLAY_POWER: Q1.1 (G), R5.2, U4.15 (PCINT30/OC2B/ICP/PD6)
- new net RF_ENABLE: R8.1
- new net VLIMIT: D7.1 (K), RV1.1, RV1.2, RV2.1, RV2.2
- no-connect marks 0 -> 4
Other:
- note added: "Keypad matrix legend"
- note added: "ROW_1,COL_1: Air Density\nROW_1,COL_2: Units Select\nROW_1,COL_3: RESET\nROW_2,COL_1: Test/Detector\nROW_2,COL_2: Measure Select\nROW_2,COL_3: Down\nROW_3,COL_2: Gain Select\nROW_3,COL_3: Up"
- moved on the sheet: J3
